Commit message: feat(raspi): add motor model that mimics firmware RPM limits
Gazebo DiffDrive tracks any requested wheel speed, while the real
firmware forces nonzero targets into 100-270 RPM. Route /cmd_vel through
a node that applies the same limits so Nav2 tuning sees real behavior.

Co-Authored-By: Claude Opus 5.5 <noreply@anthropic.com>

File: RasPi/src/agv_description/urdf/agv_gazebo.xacro (robot description, xacro)
@@ -16,6 +16,12 @@
   <xacro:wheel_friction prefix="rl"/>
   <xacro:wheel_friction prefix="rr"/>
+  <!-- Gioi han dong co GA25-370, khop SPD_RPM_MAX trong firmware (STM32/App/Inc/speed_ctrl.h).
+       Gioi han theo tung banh (va vung chet SPD_RPM_MIN) do node motor_model lo;
+       o day chi la chan tren an toan cho v va w. -->
+  <xacro:property name="wheel_rpm_max" value="270"/>
+  <xacro:property name="wheel_v_max"   value="${wheel_rpm_max * 2 * pi / 60 * wheel_radius}"/>  <!-- ~0.92 m/s -->
   <gazebo>
-    <!-- Skid-steer: DiffDrive nhan nhieu joint moi ben, 2 banh cung ben quay cung toc do -->
+    <!-- Skid-steer: DiffDrive nhan nhieu joint moi ben, 2 banh cung ben quay cung toc do.
+         Nhan lenh da qua motor_model (/model/agv/cmd_vel), khong nhan thang /cmd_vel. -->
     <plugin filename="gz-sim-diff-drive-system" name="gz::sim::systems::DiffDrive">
       <left_joint>wheel_fl_joint</left_joint>
@@ -25,7 +31,15 @@
       <wheel_separation>${effective_track}</wheel_separation>
       <wheel_radius>${wheel_radius}</wheel_radius>
+      <max_linear_velocity>${wheel_v_max}</max_linear_velocity>
+      <min_linear_velocity>${-wheel_v_max}</min_linear_velocity>
+      <max_angular_velocity>${2 * wheel_v_max / effective_track}</max_angular_velocity>
+      <min_angular_velocity>${-2 * wheel_v_max / effective_track}</min_angular_velocity>
+      <!-- Log buoc 0 -> 120 RPM (khong tai): len ~110 RPM sau 0.25 s, tuc ~1.5 m/s^2.
+           Lay 1.0 m/s^2 vi xe co tai se cham hon. -->
       <max_linear_acceleration>1.0</max_linear_acceleration>
+      <min_linear_acceleration>-1.0</min_linear_acceleration>
       <max_angular_acceleration>3.0</max_angular_acceleration>
-      <topic>/cmd_vel</topic>
+      <min_angular_acceleration>-3.0</min_angular_acceleration>
+      <topic>/model/agv/cmd_vel</topic>
       <odom_topic>/odom</odom_topic>
       <tf_topic>/tf</tf_topic>
