Commit message: feat(raspi): move lidar between tiers and add shelf lift plate
The lidar on top would be covered by the shelf deck when driving under a
shelf; between the tiers it scans at 0.12 m and also sees low pallets.

Co-Authored-By: Claude Opus 5.5 <noreply@anthropic.com>

File: RasPi/src/agv_description/urdf/agv.urdf.xacro (robot description, xacro)
@@ -3,7 +3,10 @@
   AGV kho hang: xe skid-steer 4 banh (GA25-370 x4), lidar YDLidar, IMU BNO055.
   Than xe 2 tang: 2 tam mica 30 x 30 cm cach nhau 10 cm, 4 tru oc o 4 goc.
-    - Tang 1: pin, mach, Pi, STM32 (khoi "linh kien")
-    - Tang 2: lidar
-  Frame: base_footprint (mat dat) -> base_link (tam truc banh) -> banh, laser_frame, imu_link.
+    - Tang 1: pin, mach, Pi, STM32 (khoi "linh kien"); lidar dat tren khoi linh kien, GIUA 2 tang
+    - Tang 2: co cau nang (vit me) + mat nang de chui gam va nang ke mini (kieu Amazon Kiva)
+  Lidar o giua 2 tang (mat quet ~0.12 m) vi: tren noc thi bi day ke che khi chui gam; o day
+  thi thay ca pallet thap 0.15 m. 4 tru oc che vai do -> payload_manager loc bo.
+  Frame: base_footprint (mat dat) -> base_link (tam truc banh) -> banh, laser_frame, imu_link,
+         lift_plate (khop truot lift_joint, 0 = ha, lift_stroke = nang).
   Gia tri co danh dau (*) la uoc luong - do xe that roi sua.
 -->
@@ -32,8 +35,14 @@
        effective_track moi = effective_track cu * goc_odom / goc_that. -->
   <xacro:property name="effective_track"  value="0.45"/>   <!-- hieu chinh trong sim: quay that 124 deg / odom 163 deg -->
-  <!-- Lidar tren tang 2 -->
+  <!-- Lidar giua 2 tang, dat tren khoi linh kien -->
   <xacro:property name="lidar_x"          value="0.0"/>    <!-- (*) giua mica -->
   <xacro:property name="lidar_radius"     value="0.035"/>  <!-- YDLidar X4 ~ 70 mm -->
   <xacro:property name="lidar_height"     value="0.035"/>  <!-- (*) chan de -> tam quet -->
+  <!-- Mat nang tren tang 2 (vit me + dong co nho, tu giu tai khi mat dien) -->
+  <xacro:property name="lift_plate_size"  value="0.26"/>
+  <xacro:property name="lift_plate_thickness" value="0.01"/>
+  <xacro:property name="lift_gap"         value="0.002"/>  <!-- mat nang ha het cach tang 2 -->
+  <xacro:property name="lift_stroke"      value="0.03"/>   <!-- ke mini cao gam 0.18 m: nang len ~1.7 cm khoi san -->
+  <xacro:property name="lift_speed"       value="0.02"/>   <!-- m/s, ~1.5 s cho het hanh trinh -->
   <!-- Toa do z theo base_link (truc banh) -->
   <xacro:property name="plate1_z"   value="${plate1_below_axle + plate_thickness / 2}"/>
@@ -151,5 +160,5 @@
   <xacro:wheel prefix="rl" x="${-wheelbase/2}" y="${ track_width/2}"/>
   <xacro:wheel prefix="rr" x="${-wheelbase/2}" y="${-track_width/2}"/>
-  <!-- ===================== Lidar (tang 2) ===================== -->
+  <!-- ===================== Lidar (giua 2 tang) ===================== -->
   <link name="laser_frame">
     <visual>
@@ -167,5 +176,27 @@
     <parent link="base_link"/>
     <child link="laser_frame"/>
-    <origin xyz="${lidar_x} 0 ${plate2_top + lidar_height / 2}" rpy="0 0 0"/>
+    <origin xyz="${lidar_x} 0 ${plate1_top + payload_size_z + lidar_height / 2}" rpy="0 0 0"/>
+  </joint>
+  <!-- ===================== Mat nang (tang 2) ===================== -->
+  <link name="lift_plate">
+    <visual>
+      <geometry><box size="${lift_plate_size} ${lift_plate_size} ${lift_plate_thickness}"/></geometry>
+      <material name="grey"/>
+    </visual>
+    <!-- Ten cho cam bien tiep xuc "co ke": URDF -> SDF them duoi "_collision" thanh
+         "lift_plate_collision" (ten dung trong agv_gazebo.xacro) -->
+    <collision name="lift_plate">
+      <geometry><box size="${lift_plate_size} ${lift_plate_size} ${lift_plate_thickness}"/></geometry>
+    </collision>
+    <xacro:box_inertia m="0.15" x="${lift_plate_size}" y="${lift_plate_size}" z="${lift_plate_thickness}">
+      <origin xyz="0 0 0"/>
+    </xacro:box_inertia>
+  </link>
+  <joint name="lift_joint" type="prismatic">
+    <parent link="base_link"/>
+    <child link="lift_plate"/>
+    <origin xyz="0 0 ${plate2_top + lift_gap + lift_plate_thickness / 2}" rpy="0 0 0"/>
+    <axis xyz="0 0 1"/>
+    <limit lower="0.0" upper="${lift_stroke}" effort="300" velocity="${lift_speed}"/>
   </joint>
   <!-- ===================== IMU (BNO055, tang 1) ===================== -->

File: RasPi/src/agv_description/urdf/agv_gazebo.xacro (robot description, xacro)
@@ -16,4 +16,19 @@
   <xacro:wheel_friction prefix="rl"/>
   <xacro:wheel_friction prefix="rr"/>
+  <!-- Mat nang: dem cao su, ke dat len khong truot khi xe tang toc (can mu > a/g = 0.1) -->
+  <gazebo reference="lift_plate">
+    <mu1>1.0</mu1>
+    <mu2>1.0</mu2>
+    <!-- Cam bien "co ke tren mat nang" (xe that: cong tac hanh trinh / hong ngoai) -->
+    <sensor name="lift_contact" type="contact">
+      <!-- Cam bien contact doc <topic> BEN TRONG <contact>; <topic> cap sensor bi bo qua -->
+      <contact>
+        <collision>lift_plate_collision</collision>
+        <topic>/lift/contact</topic>
+      </contact>
+      <update_rate>10</update_rate>
+      <always_on>true</always_on>
+    </sensor>
+  </gazebo>
   <!-- Gioi han dong co GA25-370, khop SPD_RPM_MAX trong firmware (STM32/App/Inc/speed_ctrl.h).
        Gioi han theo tung banh (va vung chet SPD_RPM_MIN) do node motor_model lo;
@@ -51,4 +66,19 @@
       <odom_publish_frequency>30</odom_publish_frequency>
     </plugin>
+    <!-- Co cau nang vit me: PID luc bam vi tri. lift_sim gui quy dao vi tri tang dan lift_speed
+         (vit me chay toc do gan nhu khong doi bat ke tai), PID cung + khau I giu duoc ke 3 kg (~30 N).
+         Che do use_velocity_commands da thu: khop khong chuyen dong (REPORT.md). Xe that do firmware lo. -->
+    <plugin filename="gz-sim-joint-position-controller-system"
+            name="gz::sim::systems::JointPositionController">
+      <joint_name>lift_joint</joint_name>
+      <topic>/lift/cmd_pos</topic>
+      <p_gain>10000</p_gain>
+      <i_gain>2000</i_gain>
+      <d_gain>300</d_gain>
+      <i_max>80</i_max>
+      <i_min>-80</i_min>
+      <cmd_max>300</cmd_max>
+      <cmd_min>-300</cmd_min>
+    </plugin>
     <plugin filename="gz-sim-joint-state-publisher-system" name="gz::sim::systems::JointStatePublisher">
       <topic>/joint_states</topic>
@@ -69,5 +99,6 @@
     <sensor name="lidar" type="gpu_lidar">
       <gz_frame_id>laser_frame</gz_frame_id>
-      <topic>/scan</topic>
+      <!-- /scan_raw: chua ca tru oc cua xe va chan ke dang cho -> payload_manager loc thanh /scan -->
+      <topic>/scan_raw</topic>
       <update_rate>7</update_rate>
       <always_on>true</always_on>

Commit message: feat(raspi): place simulated lidar where the CAD model puts it
Lidar moves 108 mm forward of the robot centre on M3 x 25 standoffs; the
scan plane is 119.9 mm above ground and laser_frame now sits on it.

Co-Authored-By: Claude Opus 5.5 <noreply@anthropic.com>
Claude-Session: https://claude.ai/code/session_011tprzdY2TmzTk3FoijMTum

File: RasPi/src/agv_description/urdf/agv.urdf.xacro (robot description, xacro)
@@ -3,5 +3,5 @@
   AGV kho hang: xe skid-steer 4 banh (GA25-370 x4), lidar YDLidar, IMU BNO055.
   Than xe 2 tang: 2 tam mica 30 x 30 cm cach nhau 10 cm, 4 tru oc o 4 goc.
-    - Tang 1: pin, mach, Pi, STM32 (khoi "linh kien"); lidar dat tren khoi linh kien, GIUA 2 tang
+    - Tang 1: pin, mach, Pi, STM32 (khoi "linh kien"); lidar o phia truoc tang 1 (theo CAD), GIUA 2 tang
     - Tang 2: co cau nang (vit me) + mat nang de chui gam va nang ke mini (kieu Amazon Kiva)
   Lidar o giua 2 tang (mat quet ~0.12 m) vi: tren noc thi bi day ke che khi chui gam; o day
@@ -35,8 +35,11 @@
        effective_track moi = effective_track cu * goc_odom / goc_that. -->
   <xacro:property name="effective_track"  value="0.45"/>   <!-- hieu chinh trong sim: quay that 124 deg / odom 163 deg -->
-  <!-- Lidar giua 2 tang, dat tren khoi linh kien -->
-  <xacro:property name="lidar_x"          value="0.0"/>    <!-- (*) giua mica -->
+  <!-- Lidar giua 2 tang, phia truoc xe tren 4 tru M3 x 25 (CAD/agv.FCStd, CAD/README.md).
+       laser_frame dat o mat quet; than lidar tu mat quet - lidar_below_scan toi mat quet + lidar_above_scan. -->
+  <xacro:property name="lidar_x"          value="0.108"/>  <!-- CAD: tam dau quay cach tam xe 108 mm -->
+  <xacro:property name="lidar_scan_height" value="0.1199"/> <!-- (*) CAD: mat quet cach dat 119.9 mm -->
   <xacro:property name="lidar_radius"     value="0.035"/>  <!-- YDLidar X4 ~ 70 mm -->
-  <xacro:property name="lidar_height"     value="0.035"/>  <!-- (*) chan de -> tam quet -->
+  <xacro:property name="lidar_below_scan" value="0.0384"/> <!-- (*) CAD: than cao 58.4 mm, mat quet thap hon dinh 20 mm -->
+  <xacro:property name="lidar_above_scan" value="0.020"/>  <!-- (*) -->
   <!-- Mat nang tren tang 2 (vit me + dong co nho, tu giu tai khi mat dien) -->
   <xacro:property name="lift_plate_size"  value="0.26"/>
@@ -160,15 +163,19 @@
   <xacro:wheel prefix="rl" x="${-wheelbase/2}" y="${ track_width/2}"/>
   <xacro:wheel prefix="rr" x="${-wheelbase/2}" y="${-track_width/2}"/>
-  <!-- ===================== Lidar (giua 2 tang) ===================== -->
+  <!-- ===================== Lidar (giua 2 tang, phia truoc) ===================== -->
+  <xacro:property name="lidar_len" value="${lidar_below_scan + lidar_above_scan}"/>
+  <xacro:property name="lidar_mid" value="${(lidar_above_scan - lidar_below_scan) / 2}"/>
   <link name="laser_frame">
     <visual>
-      <geometry><cylinder radius="${lidar_radius}" length="${lidar_height}"/></geometry>
+      <origin xyz="0 0 ${lidar_mid}"/>
+      <geometry><cylinder radius="${lidar_radius}" length="${lidar_len}"/></geometry>
       <material name="grey"/>
     </visual>
     <collision>
-      <geometry><cylinder radius="${lidar_radius}" length="${lidar_height}"/></geometry>
-    </collision>
-    <xacro:cylinder_inertia m="0.1" r="${lidar_radius}" h="${lidar_height}">
-      <origin xyz="0 0 0" rpy="0 0 0"/>
+      <origin xyz="0 0 ${lidar_mid}"/>
+      <geometry><cylinder radius="${lidar_radius}" length="${lidar_len}"/></geometry>
+    </collision>
+    <xacro:cylinder_inertia m="0.1" r="${lidar_radius}" h="${lidar_len}">
+      <origin xyz="0 0 ${lidar_mid}" rpy="0 0 0"/>
     </xacro:cylinder_inertia>
   </link>
@@ -176,5 +183,5 @@
     <parent link="base_link"/>
     <child link="laser_frame"/>
-    <origin xyz="${lidar_x} 0 ${plate1_top + payload_size_z + lidar_height / 2}" rpy="0 0 0"/>
+    <origin xyz="${lidar_x} 0 ${lidar_scan_height - wheel_radius}" rpy="0 0 0"/>
   </joint>
   <!-- ===================== Mat nang (tang 2) ===================== -->

Commit message: feat(raspi): adapt simulation to YDLidar X2L
430 beams per turn, 8 m range in Gazebo, AMCL and slam_toolbox;
URDF lidar pose and meshes from the CAD.

Co-Authored-By: Claude Opus 5.5 <noreply@anthropic.com>

File: RasPi/src/agv_description/urdf/agv.urdf.xacro (robot description, xacro)
@@ -1,5 +1,5 @@
 <?xml version="1.0"?>
 <!--
-  AGV kho hang: xe skid-steer 4 banh (GA25-370 x4), lidar YDLidar X4, IMU BNO055.
+  AGV kho hang: xe skid-steer 4 banh (GA25-370 x4), lidar YDLidar X2L, IMU BNO055.
   KICH THUOC VA HINH DANG LAY TU MO HINH CO KHI CAD/agv.FCStd (REPORT.md 4.16, 4.20):
     - so do: bang Params cua file CAD (CAD/export_meshes.py in ra khi chay)
@@ -9,5 +9,5 @@
     - Tang 1: DAU XE la phia PCB + Pi + camera, lidar o phia SAU (= -X cua file CAD, luoi da quay 180 deg), pin treo duoi tang 1, dong co nang NEMA17; 4 vit me T8 noi 2 tang
     - Tang 2: mat nang de chui gam va nang ke mini (kieu Amazon Kiva)
-  Lidar nam giua 2 tang, lech ve SAU 0.095 m. 4 tru oc va 4 vit me che vai do -> payload_manager loc bo.
+  Lidar nam giua 2 tang, lech ve SAU 0.092 m. 4 tru oc va 4 vit me che vai do -> payload_manager loc bo.
   Va cham (collision) van la hinh hop / tru don gian.
   Frame: base_footprint (mat dat) -> base_link (tam truc banh) -> banh, laser_frame, imu_link,
@@ -33,11 +33,11 @@
        effective_track moi = effective_track cu * goc_odom / goc_that. -->
   <xacro:property name="effective_track"  value="0.383"/>  <!-- hieu chinh trong sim: quay tai cho 2.5 rad/s, odom 2.49 / that 2.32 rad/s voi track 0.357 -->
-  <!-- Lidar YDLidar X4 (model 101.4 x 71 x 59 mm), tai bat cach mat tang 1 35 mm (tru M3 x 35),
-       tam dau quay cach tam xe 0.095 m ve phia SAU (dau xe la phia camera) -->
-  <xacro:property name="lidar_x"          value="-0.095"/>
-  <xacro:property name="lidar_scan_z"     value="0.123"/>  <!-- (*) so voi mat dat: giua dau quay (de lidar cao toi 0.113, dinh 0.133) -->
-  <xacro:property name="lidar_radius"     value="0.033"/>
-  <xacro:property name="lidar_body_z0"    value="0.074"/>  <!-- day chan lidar so voi mat dat -->
-  <xacro:property name="lidar_body_z1"    value="0.133"/>
+  <!-- Lidar YDLidar X2L (STEP GrabCAD: de 101 x 57 x 11 mm, dau quay D60 x 18 mm, dong co thoi xuong 19.4 mm duoi de),
+       day de cach mat tang 1 50 mm (3 tru M3 cai-cai 50), tam dau quay cach tam xe 0.092 m ve phia SAU -->
+  <xacro:property name="lidar_x"          value="-0.092"/>
+  <xacro:property name="lidar_scan_z"     value="0.1265"/> <!-- (*) so voi mat dat: giua dau quay (phan dung yen cao toi 0.119, dinh 0.1355) -->
+  <xacro:property name="lidar_radius"     value="0.030"/>
+  <xacro:property name="lidar_body_z0"    value="0.0871"/> <!-- day dong co lidar so voi mat dat -->
+  <xacro:property name="lidar_body_z1"    value="0.1355"/>
   <!-- Mat nang tren tang 2 (4 vit me T8 + dai GT2 + NEMA17, tu giu tai khi mat dien) -->
   <xacro:property name="lift_plate_size"  value="0.26"/>

File: RasPi/src/agv_description/urdf/agv_gazebo.xacro (robot description, xacro)
@@ -97,5 +97,5 @@
     </plugin>
   </gazebo>
-  <!-- Lidar 2D: thong so gan YDLidar X4 (360 do, ~7 Hz, 0.12-10 m) -->
+  <!-- Lidar 2D: thong so gan YDLidar X2L (360 do, 5-8 Hz, 3000 diem/s, 0.12-8 m) -->
   <gazebo reference="laser_frame">
     <sensor name="lidar" type="gpu_lidar">
@@ -109,5 +109,5 @@
         <scan>
           <horizontal>
-            <samples>720</samples>
+            <samples>430</samples>   <!-- 3000 diem/s / 7 Hz -->
             <resolution>1</resolution>
             <min_angle>-3.14159</min_angle>
@@ -122,5 +122,5 @@
           </vertical>
         </scan>
-        <!-- min 0.05 (X4 that: 0.12). Gazebo KHONG ve vat gan hon min: voi 0.12 thi tia di xuyen qua 2 tru oc
+        <!-- min 0.05 (X2L that: 0.12). Gazebo KHONG ve vat gan hon min: voi 0.12 thi tia di xuyen qua 2 tru oc
              va 2 vit me gan lidar (cach 0.075-0.112 m) nhu the chung khong ton tai. Xe that thi cac
              tru nay chan tia (lidar tra ve 0 = khong hop le). De 0.05 cho lidar mo phong thay chung,
@@ -128,5 +128,5 @@
         <range>
           <min>0.05</min>
-          <max>10.0</max>
+          <max>8.0</max>
           <resolution>0.01</resolution>
         </range>

Commit message: feat(raspi): update robot meshes and mass for the LiPo pack
Co-Authored-By: Claude Opus 5.5 <noreply@anthropic.com>

File: RasPi/src/agv_description/urdf/agv.urdf.xacro (robot description, xacro)
@@ -22,5 +22,5 @@
   <xacro:property name="plate_gap"        value="0.10"/>   <!-- mat tren tang 1 -> mat duoi tang 2 -->
   <xacro:property name="plate1_below_axle" value="0.0175"/> <!-- (*) theo ga chu L cua GA25: mat duoi tang 1 cao hon truc banh -->
-  <xacro:property name="body_mass"        value="2.6"/>    <!-- (*) ca xe tru banh va mat nang: 2 mica ~1.0, 5 dong co ~0.7, pin, mach, lidar -->
+  <xacro:property name="body_mass"        value="2.8"/>    <!-- (*) ca xe tru banh va mat nang: 2 mica ~1.0, 5 dong co ~0.7, pin LiPo 3S 5200mAh ~0.4, mach, lidar -->
   <!-- Banh "65 mm": duong kinh ngoai thuc 68 mm (model banh) -->
   <xacro:property name="wheel_radius"     value="0.034"/>
