File: PCB/agv_mainboard.kicad_pcb (KiCad board)
At the start: 2 copper layers, 150 x 120 mm, 61 parts, among them J1 BAT_3S, J10 DISCOVERY_P1, J11 DISCOVERY_P2, J2 SW_PWR, J20 MOTOR1_PH2.0, J21 MOTOR2_PH2.0, J22 MOTOR3_PH2.0, J23 MOTOR4_PH2.0, J3 CHARGE, J30 STEPPER_XH, J31 LIMIT_UP, J32 LIMIT_DOWN, J4 PI_BUCK_OUT, J40 I2C_SPARE, J41 UART_PI, J5 ESTOP_NC, Q1 IRF4905, Q2 BC547, U1 INA169_5A, U2 XL4015_5V, U3 LD1117V33, U4 TB6612FNG_M1_M2, U5 TB6612FNG_M3_M4, U6 A4988, U7 GY-BNO055

Commit message: wip: local CAD meshes, URDF, PCB and STM32 changes
Parts:
- removed C1, C10, C11, C7: 100nF, Capacitor_THT:C_Disc_D5.0mm_W2.5mm_P5.00mm
- removed C2: 1000uF/25V, Capacitor_THT:CP_Radial_D10.0mm_P5.00mm
- removed C3, C8, C9: 100uF/25V, Capacitor_THT:CP_Radial_D6.3mm_P2.50mm
- removed C4: 10uF, Capacitor_THT:CP_Radial_D5.0mm_P2.00mm
- removed D3: LED_VBAT, LED_THT:LED_D3.0mm
- removed D5: LED_5V, LED_THT:LED_D3.0mm
- removed R1: 100k, Resistor_THT:R_Axial_DIN0207_L6.3mm_D2.5mm_P10.16mm_Horizontal
- removed R10, R2, R4: 10k, Resistor_THT:R_Axial_DIN0207_L6.3mm_D2.5mm_P10.16mm_Horizontal
- removed R3: 39k, Resistor_THT:R_Axial_DIN0207_L6.3mm_D2.5mm_P10.16mm_Horizontal
- removed R7: 4.7k, Resistor_THT:R_Axial_DIN0207_L6.3mm_D2.5mm_P10.16mm_Horizontal
- removed R9: 1k, Resistor_THT:R_Axial_DIN0207_L6.3mm_D2.5mm_P10.16mm_Horizontal
- F1: value 5A -> 8A
- J4: value PI_BUCK_OUT -> PI_BUCK_5V10A
- U1: value INA169_5A -> INA219; footprint agv_modules:INA169_Module -> agv_modules:INA219_Module
- moved J4 268.4 mm to (316.2, 184.7)
- moved J23 261.7 mm to (323.8, 247.6)
- moved J22 260.8 mm to (304.9, 247.6)
- moved J41 251.4 mm to (236.2, 297.1)
- moved U7 239.7 mm to (216.8, 296.1)
- moved D1 232.4 mm to (287.6, 137.6), turned to 90 degrees
- moved J3 224.4 mm to (276.2, 124.0)
- moved D6 222.6 mm to (270.1, 238.7), turned to 90 degrees
- moved U3 218.5 mm to (276.2, 184.6)
- moved J40 218.5 mm to (226.4, 297.2)
- moved R13 215.4 mm to (263.8, 231.5), turned to 180 degrees
- moved C14 210.8 mm to (316.9, 278.6)
- moved J2 210.3 mm to (263.6, 128.5), turned to 90 degrees
- moved D4 210.2 mm to (273.7, 213.9), turned to 180 degrees
- moved C5 209.7 mm to (287.0, 181.2)
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Connections:
- net +5V_DISC renamed /+5V_DISC
- net BAT_FUSED renamed /BAT_FUSED
- net BAT_IN renamed /BAT_IN
- net BUZZER renamed /BUZZER
- net BUZ_B renamed /BUZ_B
- net BUZ_C renamed /BUZ_C
- net CHG_IN renamed /CHG_IN
- net ENC1_A renamed /ENC1_A
- net ENC1_B renamed /ENC1_B
- net ENC2_A renamed /ENC2_A
- net ENC2_B renamed /ENC2_B
- net ENC3_A renamed /ENC3_A
- net ENC3_B renamed /ENC3_B
- net ENC4_A renamed /ENC4_A
- net ENC4_B renamed /ENC4_B
- net ESTOP_SENSE renamed /ESTOP_SENSE
- net LED_VMOT renamed /LED_VMOT
- net LIFT_DIR renamed /LIFT_DIR
- net LIFT_SW_DOWN renamed /LIFT_SW_DOWN
- net LIFT_SW_UP renamed /LIFT_SW_UP
- net M1_IN2 renamed /M1_IN2
- net M2_IN1 renamed /M2_IN1
- net M2_IN2 renamed /M2_IN2
- net M2_PWM renamed /M2_PWM
- net M3_IN1 renamed /M3_IN1
- net M3_IN2 renamed /M3_IN2
- net M3_PWM renamed /M3_PWM
- net M4_IN1 renamed /M4_IN1
- net M4_IN2 renamed /M4_IN2
- net M4_PWM renamed /M4_PWM
- net MOT1_N renamed /MOT1_N
- net MOT1_P renamed /MOT1_P
- net MOT2_N renamed /MOT2_N
- net MOT2_P renamed /MOT2_P
- net MOT3_N renamed /MOT3_N
- net MOT3_P renamed /MOT3_P
- net MOT4_N renamed /MOT4_N
- net MOT4_P renamed /MOT4_P
- net MOTOR_STBY renamed /MOTOR_STBY
- net MS1 renamed /MS1
- net MS2 renamed /MS2
- net MS3 renamed /MS3
- net STEP_1A renamed /STEP_1A
- net STEP_1B renamed /STEP_1B
- net STEP_2A renamed /STEP_2A
- net STEP_2B renamed /STEP_2B
- net UART_RX renamed /UART_RX
- net UART_TX renamed /UART_TX
- net VBAT_PROT renamed /VBAT_PROT
- net VMOT renamed /VMOT
- J10 pad 10: (no net) -> unconnected-(J10-Pin_10-Pad10)
- J10 pad 11: VBAT_SENSE -> unconnected-(J10-Pin_11-Pad11)
- J10 pad 12: (no net) -> unconnected-(J10-Pin_12-Pad12)
- J10 pad 15: (no net) -> unconnected-(J10-Pin_15-Pad15)
- J10 pad 16: (no net) -> unconnected-(J10-Pin_16-Pad16)
- J10 pad 17: (no net) -> unconnected-(J10-Pin_17-Pad17)
- J10 pad 18: (no net) -> unconnected-(J10-Pin_18-Pad18)
- J10 pad 19: (no net) -> unconnected-(J10-Pin_19-Pad19)
- J10 pad 20: (no net) -> unconnected-(J10-Pin_20-Pad20)
- J10 pad 21: (no net) -> unconnected-(J10-Pin_21-Pad21)
- J10 pad 22: (no net) -> unconnected-(J10-Pin_22-Pad22)
- J10 pad 24: (no net) -> unconnected-(J10-Pin_24-Pad24)
- J10 pad 25: M1_IN1 -> unconnected-(J10-Pin_25-Pad25)
- J10 pad 27: M1_PWM -> unconnected-(J10-Pin_27-Pad27)
- J10 pad 3: (no net) -> unconnected-(J10-Pin_3-Pad3)
- J10 pad 34: (no net) -> unconnected-(J10-Pin_34-Pad34)
- J10 pad 36: (no net) -> /M1_IN1
- J10 pad 38: (no net) -> /M1_PWM
- J10 pad 4: (no net) -> unconnected-(J10-Pin_4-Pad4)
- J10 pad 40: (no net) -> unconnected-(J10-Pin_40-Pad40)
- J10 pad 42: (no net) -> unconnected-(J10-Pin_42-Pad42)
- J10 pad 44: (no net) -> unconnected-(J10-Pin_44-Pad44)
- J10 pad 45: (no net) -> unconnected-(J10-Pin_45-Pad45)
- J10 pad 46: (no net) -> unconnected-(J10-Pin_46-Pad46)
- J10 pad 47: (no net) -> unconnected-(J10-Pin_47-Pad47)
- J10 pad 48: (no net) -> unconnected-(J10-Pin_48-Pad48)
- J10 pad 6: (no net) -> unconnected-(J10-Pin_6-Pad6)
- J10 pad 7: ISENSE -> unconnected-(J10-Pin_7-Pad7)
- J10 pad 8: (no net) -> unconnected-(J10-Pin_8-Pad8)
- J10 pad 9: (no net) -> unconnected-(J10-Pin_9-Pad9)
- J11 pad 10: (no net) -> unconnected-(J11-Pin_10-Pad10)
- J11 pad 11: LIFT_EN -> /LIFT_STEP
- J11 pad 12: (no net) -> unconnected-(J11-Pin_12-Pad12)
- J11 pad 14: LIFT_STEP -> unconnected-(J11-Pin_14-Pad14)
- J11 pad 15: (no net) -> /LIFT_EN
- J11 pad 16: (no net) -> unconnected-(J11-Pin_16-Pad16)
- J11 pad 17: (no net) -> unconnected-(J11-Pin_17-Pad17)
- J11 pad 18: (no net) -> unconnected-(J11-Pin_18-Pad18)
- J11 pad 19: (no net) -> unconnected-(J11-Pin_19-Pad19)
- J11 pad 20: (no net) -> unconnected-(J11-Pin_20-Pad20)
- J11 pad 21: (no net) -> unconnected-(J11-Pin_21-Pad21)
- J11 pad 22: (no net) -> unconnected-(J11-Pin_22-Pad22)
- J11 pad 27: (no net) -> unconnected-(J11-Pin_27-Pad27)
- J11 pad 29: (no net) -> unconnected-(J11-Pin_29-Pad29)
- J11 pad 31: (no net) -> unconnected-(J11-Pin_31-Pad31)
- J11 pad 32: (no net) -> unconnected-(J11-Pin_32-Pad32)
- J11 pad 33: (no net) -> unconnected-(J11-Pin_33-Pad33)
- J11 pad 35: (no net) -> unconnected-(J11-Pin_35-Pad35)
- J11 pad 37: (no net) -> unconnected-(J11-Pin_37-Pad37)
- J11 pad 38: (no net) -> /IMU_RST
- J11 pad 39: (no net) -> unconnected-(J11-Pin_39-Pad39)
- J11 pad 41: (no net) -> unconnected-(J11-Pin_41-Pad41)
- J11 pad 42: (no net) -> unconnected-(J11-Pin_42-Pad42)
- J11 pad 43: I2C_SCL -> /I2C_SCL
- J11 pad 44: (no net) -> unconnected-(J11-Pin_44-Pad44)
- J11 pad 45: (no net) -> unconnected-(J11-Pin_45-Pad45)
- J11 pad 46: I2C_SDA -> /I2C_SDA
- J11 pad 5: (no net) -> unconnected-(J11-Pin_5-Pad5)
- J11 pad 6: (no net) -> unconnected-(J11-Pin_6-Pad6)
- J11 pad 7: (no net) -> unconnected-(J11-Pin_7-Pad7)
- J11 pad 8: (no net) -> unconnected-(J11-Pin_8-Pad8)
- J11 pad 9: (no net) -> unconnected-(J11-Pin_9-Pad9)
- J2 pad 2: VBAT_SW -> /VBAT_SW
- J4 pad 1: VBAT -> /VBAT
- J40 pad 3: I2C_SCL -> /I2C_SCL
- J40 pad 4: I2C_SDA -> /I2C_SDA
- J5 pad 1: VBAT -> /VBAT
- Q1 pad 1: Q1_G -> GND
- R11 pad 2: LIFT_EN -> /LIFT_EN
- U1 pad 1: VBAT_SW -> +3V3
- U1 pad 2: VBAT -> GND
- U1 pad 3: +5V -> /I2C_SCL
- U1 pad 4: GND -> /I2C_SDA
- U1 pad 5: ISENSE -> /VBAT
- U2 pad 1: VBAT -> /VBAT
- U4 pad 11: M1_IN1 -> /M1_IN1
- U4 pad 9: M1_PWM -> /M1_PWM
- U6 pad 15: LIFT_STEP -> /LIFT_STEP
- U6 pad 9: LIFT_EN -> /LIFT_EN
- U7 pad 3: I2C_SCL -> /I2C_SCL
- U7 pad 4: I2C_SDA -> /I2C_SDA
- U7 pad 5: (no net) -> GND
- U7 pad 6: (no net) -> unconnected-(U7-INT-Pad6)
- U7 pad 7: (no net) -> unconnected-(U7-BOOT-Pad7)
- U7 pad 8: (no net) -> /IMU_RST
Other:
- board size 150 x 120 mm -> 150 x 125 mm
