File: PCB/agv_mainboard.kicad_pcb (KiCad board)
At the start: 2 copper layers, 150 x 125 mm, 43 parts, among them J1 BAT_3S, J10 DISCOVERY_P1, J11 DISCOVERY_P2, J2 SW_PWR, J20 MOTOR1_PH2.0, J21 MOTOR2_PH2.0, J22 MOTOR3_PH2.0, J23 MOTOR4_PH2.0, J3 CHARGE, J30 STEPPER_XH, J31 LIMIT_UP, J32 LIMIT_DOWN, J4 PI_BUCK_5V10A, J40 I2C_SPARE, J41 UART_PI, J5 ESTOP_NC, Q1 IRF4905, Q2 BC547, U1 INA219, U2 XL4015_5V, U3 LD1117V33, U4 TB6612FNG_M1_M2, U5 TB6612FNG_M3_M4, U6 A4988, U7 GY-BNO055

Commit message: feat(pcb): route mainboard on two layers with JLCPCB rules
DRC with schematic parity: 0 violations, 0 unconnected pads.

Co-Authored-By: Claude Opus 5.5 <noreply@anthropic.com>
Parts:
- added H1: MountingHole_3.2mm_M3, MountingHole_3.2mm_M3, F.Cu at (54.0, 54.0)
- added H2: MountingHole_3.2mm_M3, MountingHole_3.2mm_M3, F.Cu at (196.0, 54.0)
- added H3: MountingHole_3.2mm_M3, MountingHole_3.2mm_M3, F.Cu at (54.0, 171.0)
- added H4: MountingHole_3.2mm_M3, MountingHole_3.2mm_M3, F.Cu at (196.0, 171.0)
- moved J4 280.7 mm to (61.5, 66.5), turned to 0 degrees
- moved J23 258.1 mm to (78.5, 167.4)
- moved J22 256.3 mm to (61.5, 167.4)
- moved D1 223.3 mm to (64.9, 121.1)
- moved U5 221.1 mm to (72.8, 105.6)
- moved J3 220.7 mm to (55.5, 125.0), turned to 90 degrees
- moved D6 213.6 mm to (76.1, 149.3), turned to 0 degrees
- moved JP1 212.3 mm to (95.8, 133.4)
- moved C12 211.9 mm to (96.2, 140.4)
- moved R11 211.4 mm to (106.1, 142.5)
- moved J2 208.3 mm to (55.5, 138.0)
- moved D2 207.6 mm to (118.6, 94.6)
- moved U6 204.7 mm to (71.6, 142.3)
- moved U4 197.8 mm to (97.8, 105.6), turned to 0 degrees
- moved R13 197.5 mm to (81.1, 156.5), turned to 0 degrees
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Routing:
- net +3V3: track 0.00 -> 324.6 mm, vias 0 -> 1
- net /I2C_SDA: track 0.00 -> 237.2 mm, vias 0 -> 3
- net /I2C_SCL: track 0.00 -> 224.5 mm, vias 0 -> 3
- net +5V: track 0.00 -> 183.8 mm
- net /ENC3_B: track 0.00 -> 169.5 mm, vias 0 -> 1
- net /ENC3_A: track 0.00 -> 155.0 mm, vias 0 -> 2
- net /VMOT: track 0.00 -> 153.5 mm
- net /ENC1_B: track 0.00 -> 147.7 mm, vias 0 -> 2
- net /LIFT_EN: track 0.00 -> 146.6 mm, vias 0 -> 3
- net /ENC1_A: track 0.00 -> 140.5 mm, vias 0 -> 2
- net /LIFT_STEP: track 0.00 -> 134.0 mm, vias 0 -> 1
- net /LIFT_DIR: track 0.00 -> 126.7 mm
- net /ENC4_B: track 0.00 -> 116.8 mm
- net /ENC4_A: track 0.00 -> 115.7 mm
- net /ESTOP_SENSE: track 0.00 -> 112.0 mm, vias 0 -> 2
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- added copper zone on B.Cu, net GND
- added copper zone on F.Cu, net GND

Commit message: fix(pcb): face terminal blocks outward and take battery via XT60
Wire entries of J2, J3, J5 now face the left edge and J4 the top edge.
J1 becomes an XT60PW-M jack for a LiPo pack. Rerouted: DRC with
schematic parity 0/0/0.

Co-Authored-By: Claude Opus 5.5 <noreply@anthropic.com>
Parts:
- J1: value BAT_3S -> XT60_LIPO_3S; footprint TerminalBlock:TerminalBlock_MaiXu_MX126-5.0-02P_1x02_P5.00mm -> agv_modules:XT60PW-M_Battery_Pin1Plus
- moved J1 17.8 mm to (67.4, 72.4), turned to 90 degrees
- moved J4 12.5 mm to (66.0, 54.9), turned to 180 degrees
- moved J2 4.50 mm to (55.4, 133.5), turned to -90 degrees
- moved J3 4.50 mm to (55.4, 120.5), turned to -90 degrees
- moved J5 4.50 mm to (55.4, 107.5), turned to -90 degrees
Routing:
- net /MOT1_P: track 105.3 -> 56.8 mm, vias 2 -> 0
- net /MOT2_P: track 56.9 -> 85.1 mm, vias 0 -> 5
- net GND: track 20.4 -> 0.00 mm, vias 380 -> 0
- net /MOT2_N: track 83.0 -> 65.0 mm, vias 2 -> 1
- net /ENC1_A: track 140.5 -> 123.2 mm, vias 2 -> 1
- net /BAT_FUSED: track 12.6 -> 28.9 mm
- net /LIFT_EN: track 146.6 -> 130.4 mm, vias 3 -> 2
- net /M3_PWM: track 70.8 -> 56.1 mm
- net /LIFT_DIR: track 126.7 -> 138.9 mm, vias 0 -> 2
- net /STEP_1A: track 67.8 -> 79.2 mm, vias 0 -> 1
- net /BAT_IN: track 35.5 -> 24.2 mm
- net +5V: track 183.8 -> 195.1 mm, vias 0 -> 1
- net /IMU_RST: track 90.8 -> 79.6 mm, vias 1 -> 2
- net /I2C_SCL: track 224.5 -> 235.1 mm, vias 3 -> 5
- net /ENC4_A: track 115.7 -> 126.0 mm, vias 0 -> 1
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