File: PCB/agv_mainboard.kicad_sch (KiCad schematic)
At the start: 48 parts, among them J1 BAT_3S, J10 DISCOVERY_P1, J11 DISCOVERY_P2, J2 SW_PWR, J20 MOTOR1_PH2.0, J21 MOTOR2_PH2.0, J22 MOTOR3_PH2.0, J23 MOTOR4_PH2.0, J3 CHARGE, J30 STEPPER_XH, J31 LIMIT_UP, J32 LIMIT_DOWN, J4 PI_BUCK_OUT, J40 I2C_SPARE, J41 UART_PI, J5 ESTOP_NC, Q1 IRF4905, Q2 BC547, U1 INA169_5A, U2 XL4015_5V, U3 LD1117V33, U4 TB6612FNG_M1_M2, U5 TB6612FNG_M3_M4, U6 A4988, U7 GY-BNO055

Commit message: wip: local CAD meshes, URDF, PCB and STM32 changes
Parts:
- removed C1, C7: 100nF, Capacitor_THT:C_Disc_D5.0mm_W2.5mm_P5.00mm, symbol Device:C
- removed R2, R4: 10k, Resistor_THT:R_Axial_DIN0207_L6.3mm_D2.5mm_P10.16mm_Horizontal, symbol Device:R
- removed R3: 39k, Resistor_THT:R_Axial_DIN0207_L6.3mm_D2.5mm_P10.16mm_Horizontal, symbol Device:R
- removed U1: INA169_5A, agv_modules:INA169_Module, symbol agv_modules:INA169_Module
- added U1: INA219, agv_modules:INA219_Module, symbol agv_modules:INA219_Module
- F1: value 5A -> 8A
- J4: value PI_BUCK_OUT -> PI_BUCK_5V10A
Connections:
- net +3V3: now also U1.1 (VCC)
- net GND: now also U7.5 (ADD), U1.2 (GND)
- net I2C_SCL: now also U1.3 (SCL)
- net I2C_SDA: now also U1.4 (SDA)
- net LIFT_EN: now also J11.15 (Pin_15); no longer J11.11 (Pin_11)
- net LIFT_STEP: now also J11.11 (Pin_11); no longer J11.14 (Pin_14)
- net M1_IN1: now also J10.36 (Pin_36); no longer J10.25 (Pin_25)
- net M1_PWM: now also J10.38 (Pin_38); no longer J10.27 (Pin_27)
- net VBAT: now also U1.5 (VIN-)
- net VBAT_SW: now also U1.6 (VIN+)
- net IMU_RST: now reaches J11.38 (Pin_38)
- net IMU_RST: now also U7.8 (RST)
- net ISENSE: no longer names the net of J10.7 (Pin_7)
- net VBAT_SENSE: no longer names the net of J10.11 (Pin_11)
- no-connect marks 58 -> 57
Other:
- note added: "1. NGUỒN VÀO - BẢO VỆ - SẠC"
- note added: "2. ĐO DÒNG VÀ ÁP PIN (INA219)"
- note added: "BZ1: còi 5 V báo pin yếu, dừng khẩn, sự cố. D6: dập xung ngược của còi."
- note added: "J1: đầu vào pin 3S (9 - 12.6 V). F1: cầu chì 8 A cho toàn bộ xe, kể cả Pi."
- note added: "J3: tiếp điểm sạc 12.6 V, sạc được cả khi công tắc nguồn mở. D1: không cho áp pin ra tiếp điểm."
- note added: "J4: cấp điện áp pin cho buck 5 V / 10 A gắn ngoài của Raspberry Pi. U2: buck XL4015 hạ xuống 5 V cho mạch logic (module đã có sẵn tụ lọc đầu vào và đầu ra)."
- note added: "Shunt gốc 0.1 ohm chỉ đo 3.2 A: thay bằng 0.02 ohm 2 W (đo tới 16 A)."
- note added: "U1: INA219 đo dòng và điện áp pin của cả xe (kể cả Pi),"
- note added: "U3: ổn áp 3.3 V cho encoder, INA219 và logic driver. C5: tụ bắt buộc ở đầu ra U3. D2: không cho USB của Discovery cấp ngược vào đường 5 V."
- note added: "U7: IMU, I2C 0x28 (ADD nối mass), MCU điều khiển RST. J40: I2C dự phòng."
- note added: "gửi về MCU qua I2C (0x40). Cấp 3.3 V để mức I2C hợp với BNO055."
- note removed: "1. NGUỒN VÀO - BẢO VỆ"
- note removed: "2. ĐO DÒNG - ĐO ÁP PIN"
- note removed: "BZ1: còi 5 V. D6: dập xung ngược của còi."
- note removed: "J1: đầu vào pin 3S (9 - 12.6 V). F1: cầu chì 5 A bảo vệ quá dòng."
- note removed: "J3: tiếp điểm sạc. D1: không cho điện áp pin ra tiếp điểm sạc."
- note removed: "J4: xuất điện áp pin cho buck ngoài của Raspberry Pi. U2: buck XL4015 hạ xuống 5 V cho mạch logic (module đã có sẵn tụ lọc đầu vào và đầu ra)."
- note removed: "R2: giảm còn 0.5 V/A cho vừa ADC 3 V. C1: lọc nhiễu."
- note removed: "R3, R4: chia áp pin về 2.6 V để đo. C7: lọc nhiễu."
- note removed: "U1: đo dòng pin, ngõ ra điện áp 1 V/A."
- note removed: "U3: ổn áp 3.3 V cho encoder và logic driver. C5: tụ bắt buộc ở đầu ra U3. D2: không cho USB của Discovery cấp ngược vào đường 5 V."
- note removed: "U7: IMU 9 trục. J40: I2C dự phòng. J41: UART sang Raspberry Pi."
