File: PCB/agv_mainboard.kicad_sch (KiCad schematic)
At the start: 43 parts, among them J1 BAT_3S, J10 DISCOVERY_P1, J11 DISCOVERY_P2, J2 SW_PWR, J20 MOTOR1_PH2.0, J21 MOTOR2_PH2.0, J22 MOTOR3_PH2.0, J23 MOTOR4_PH2.0, J3 CHARGE, J30 STEPPER_XH, J31 LIMIT_UP, J32 LIMIT_DOWN, J4 PI_BUCK_5V10A, J40 I2C_SPARE, J41 UART_PI, J5 ESTOP_NC, Q1 IRF4905, Q2 BC547, U1 INA219, U2 XL4015_5V, U3 LD1117V33, U4 TB6612FNG_M1_M2, U5 TB6612FNG_M3_M4, U6 A4988, U7 GY-BNO055

Commit message: fix(pcb): face terminal blocks outward and take battery via XT60
Wire entries of J2, J3, J5 now face the left edge and J4 the top edge.
J1 becomes an XT60PW-M jack for a LiPo pack. Rerouted: DRC with
schematic parity 0/0/0.

Co-Authored-By: Claude Opus 5.5 <noreply@anthropic.com>
Parts:
- J1: value BAT_3S -> XT60_LIPO_3S; footprint TerminalBlock:TerminalBlock_MaiXu_MX126-5.0-02P_1x02_P5.00mm -> agv_modules:XT60PW-M_Battery_Pin1Plus
Changed lines of the file:
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@@
 			)
 		)
-		(property "Value" "BAT_3S"
+		(property "Value" "XT60_LIPO_3S"
 			(at 27.94 51.46 0)
 			(show_name no)
@@
 			)
 		)
-		(property "Footprint" "TerminalBlock:TerminalBlock_MaiXu_MX126-5.0-02P_1x02_P5.00mm"
+		(property "Footprint" "agv_modules:XT60PW-M_Battery_Pin1Plus"
 			(at 27.94 45.72 0)
 			(hide yes)
@@
 			)
 		)
-		(property "Datasheet" ""
+		(property "Datasheet" "https://www.tme.eu/Document/b13629717d44ae038681dba08d18c0b6/XT60PW-M.pdf"
 			(at 27.94 45.72 0)
 			(hide yes)
@@
 			)
 		)
-		(property "Description" "Generic screw terminal, single row, 01x02, script generated (kicad-library-utils/schlib/autogen/connector/)"
+		(property "Description" "Jack XT60 duc han mach nam ngang, nguon vao tu pin LiPo 3S (chan 1 = +)"
 			(at 27.94 45.72 0)
 			(hide yes)
